Commit message: Added visualization of pinger bearing and a few other tweaks.

File: models/cobalt.urdf (robot description, URDF)
Before this commit: robot robosub_cobalt, 19 links, 18 joints
Links:
- removed link base_link
- removed link left_camera
- added link cobalt
- added link left_cam, mass 0.73; collision cylinder length=0.15 radius=0.0405; visual cylinder length=0.15 radius=0.0405
Joints:
- joint frame_base: parent base_link -> cobalt
- joint left_camera_frame: child left_camera -> left_cam
